Commit message: Use model directive to build environment

File: sandbox/planar_iiwa14_one_sphere.urdf (robot description, URDF)
Before this commit: robot iiwa14, 10 links, 9 joints
Links:
- link iiwa_link_0: geometry visual mesh filename=package://drake/manipulation/models/iiwa_description/meshes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
- link iiwa_link_1: geometry visual mesh filename=package://drake/manipulation/models/iiwa_description/meshes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
- link iiwa_link_2: geometry visual mesh filename=package://drake/manipulation/models/iiwa_description/meshes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; visual mesh filename=package://drake/manipulation/models/iiwa_description/meshes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
- link iiwa_link_3: geometry visual mesh filename=package://drake/manipulation/models/iiwa_description/meshes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; visual mesh filename=package://drake/manipulation/models/iiwa_description/meshes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
- link iiwa_link_4: geometry visual mesh filename=package://drake/manipulation/models/iiwa_description/meshes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; visual mesh filename=package://drake/manipulation/models/iiwa_description/meshes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
- link iiwa_link_5: geometry visual mesh filename=package://drake/manipulation/models/iiwa_description/meshes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; visual mesh filename=package://drake/manipulation/models/iiwa_description/meshes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
- link iiwa_link_6: geometry visual mesh filename=package://drake/manipulation/models/iiwa_description/meshes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; visual mesh filename=package://drake/manipulation/models/iiwa_description/meshes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
- link iiwa_link_7: geometry collision box size=.12 .12 .12; visual mesh filename=package://drake/manipulation/models/iiwa_description/meshes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
