Commit message: collision checking working

File: sandbox/planar2dof.urdf (robot description, URDF)
Before this commit: robot planar2dof_robot, 3 links, 2 joints
Links:
- added link box1; collision box size=0.4 0.1 1.8; visual box size=0.4 0.1 1.8
- added link box2; collision box size=0.4 0.1 2.0; visual box size=0.4 0.1 2.0
- added link box3; collision box size=0.4 0.1 1.8; visual box size=0.4 0.1 1.8
- added link box4; collision box size=0.4 0.1 2.0; visual box size=0.4 0.1 2.0
- added link link1viz; visual box size=0.04 0.04 1.0
- added link link2viz; visual box size=0.04 0.04 0.8
- added link link3, mass 1; collision box size=0.1 0.1 0.8; visual box size=0.1 0.1 0.8
- added link link3viz; visual box size=0.04 0.04 0.8
- link link1: geometry collision box size=0.1 0.1 0.8; visual box size=0.1 0.1 0.8
- link link2: geometry collision box size=0.1 0.1 0.8; visual box size=0.1 0.1 0.8
Joints:
- added joint joint3: type revolute, parent base, child link3, origin xyz=0 -1.5 0.1 rpy=0 0 0, axis -1 0 0, limit lower=0.0 upper=1.5707
- added joint joint4: type fixed, parent base, child box1, origin xyz=0 -0.75 -0.05 rpy=1.5707 0 0
- added joint joint5: type fixed, parent base, child box2, origin xyz=0 0.2 1.0 rpy=0 0 0
- added joint joint6: type fixed, parent base, child box3, origin xyz=0 -0.75 2.0 rpy=1.5707 0 0
- added joint joint7: type fixed, parent base, child box4, origin xyz=0 -1.7 1.0 rpy=0 0 0
- added joint jointv1: type fixed, parent link1, child link1viz, origin xyz=0 0 0 rpy=0 0 0
- added joint jointv2: type fixed, parent link2, child link2viz, origin xyz=0 0 0 rpy=0 0 0
- added joint jointv3: type fixed, parent link3, child link3viz, origin xyz=0 0 -0.2 rpy=0 0 0
