Commit message: collision checking not working

File: sandbox/assets/planar1dof.urdf (robot description, URDF)
Before this commit: robot planar1dof_robot, 3 links, 2 joints
Joints:
- joint joint1: limit lower=0.0 upper=1.5707 -> lower=-1.5707 upper=1.5707

File: sandbox/assets/planar2dof.urdf (robot description, URDF)
Before this commit: robot planar2dof_robot, 5 links, 4 joints
Joints:
- joint joint1: limit lower=0.0 upper=1.5707 -> (none)
- joint joint2: limit lower=0.0 upper=1.5707 -> (none)
