Commit message: collision checking not working

File: sandbox/assets/box.urdf (robot description, URDF)
Before this commit: robot box_scene, 5 links, 4 joints
Joints:
- removed joint joint5
- removed joint joint6
- removed joint joint7
- added joint joint1: type fixed, parent base, child box1, origin xyz=0 -0.75 -0.05 rpy=1.5707 0 0
- added joint joint2: type fixed, parent base, child box2, origin xyz=0 0.2 1.0 rpy=0 0 0
- added joint joint3: type fixed, parent base, child box3, origin xyz=0 -0.75 2.0 rpy=1.5707 0 0
- joint joint4: child box1 -> box4; origin xyz=0 -0.75 -0.05 rpy=1.5707 0 0 -> xyz=0 -1.7 1.0 rpy=0 0 0

File: sandbox/assets/planar1dof.urdf (robot description, URDF)
Before this commit: robot planar1dof_robot, 3 links, 2 joints
Joints:
- joint joint1: origin xyz=0 -1.5 0.0 rpy=0 0 0 -> xyz=0 0 0 rpy=0 0 0

Commit message: planar example working

File: sandbox/assets/box.urdf (robot description, URDF)
Before this commit: robot box_scene, 5 links, 4 joints
Joints:
- removed joint joint1
- removed joint joint2
- removed joint joint3
- removed joint joint4
- added joint jbox1: type fixed, parent base, child box1, origin xyz=0 -0.75 -0.05 rpy=1.5707 0 0
- added joint jbox2: type fixed, parent base, child box2, origin xyz=0 0.2 1.0 rpy=0 0 0
- added joint jbox3: type fixed, parent base, child box3, origin xyz=0 -0.75 2.0 rpy=1.5707 0 0
- added joint jbox4: type fixed, parent base, child box4, origin xyz=0 -1.7 1.0 rpy=0 0 0

File: sandbox/assets/doublerob.urdf (robot description, URDF)
Before this commit: robot planar2dof_robot, 5 links, 4 joints
Links:
- added link linka, mass 1; collision box size=0.1 0.1 0.8; visual box size=0.1 0.1 0.8
- added link linkaviz; visual box size=0.04 0.04 0.8
Joints:
- added joint jointa: type revolute, parent base, child linka, origin xyz=0 -1.5 0 rpy=0 0 0, axis 1 0 0
- added joint jointva: type fixed, parent linka, child linkaviz, origin xyz=0 0 -0.2 rpy=0 0 0

Commit message: iris running in 2d example

File: sandbox/assets/box.urdf (robot description, URDF)
Before this commit: robot box_scene, 5 links, 4 joints
Joints:
- joint jbox2: origin xyz=0 0.2 1.0 rpy=0 0 0 -> xyz=0 0.6 1.0 rpy=0 0 0

File: sandbox/assets/doublerob.urdf (robot description, URDF)
Before this commit: robot planar2dof_robot, 7 links, 6 joints
Joints:
- joint jointa: origin xyz=0 -1.5 0 rpy=0 0 0 -> xyz=0 -1.5 0.4 rpy=0 0 0

Commit message: 2d iris working

File: sandbox/assets/box.urdf (robot description, URDF)
Before this commit: robot box_scene, 5 links, 4 joints
Links:
- link box1: geometry collision box size=0.4 0.1 2.4; visual box size=0.4 0.1 2.4
- link box3: geometry collision box size=0.4 0.1 2.4; visual box size=0.4 0.1 2.4
Joints:
- joint jbox1: origin xyz=0 -0.75 -0.05 rpy=1.5707 0 0 -> xyz=0 -0.55 -0.05 rpy=1.5707 0 0
- joint jbox3: origin xyz=0 -0.75 2.0 rpy=1.5707 0 0 -> xyz=0 -0.55 2.0 rpy=1.5707 0 0

File: sandbox/assets/doublerob.urdf (robot description, URDF)
Before this commit: robot planar2dof_robot, 7 links, 6 joints
Links:
- added link linkbaviz; visual box size=0.04 0.04 0.4
Joints:
- added joint jointvba: type fixed, parent base, child linkbaviz, origin xyz=0 -1.5 0.0 rpy=0 0 0
